File: EURO SMD 2 boards Function Generator.kicad_pcb (KiCad board)
At the start: 2 copper layers, 124.1 x 110.8 mm, 107 parts, among them J1 Synth_power_2x5, J2 Conn_01x10_Male, Q1 2N3904, Q2 2N3904, SW1 SW_SPDT, SW2 SW_DPDT_x2, SW3 SW_Push, U1 TL074, U2 TL074, U3 TL074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

Commit message: Add files via upload
Parts:
- moved R45 91.0 mm to (78.0, 95.2), turned to -90 degrees
- moved R46 86.7 mm to (80.5, 95.2), turned to 90 degrees
- moved R22 6.68 mm to (115.0, 103.5)
- moved R7 4.85 mm to (165.6, 88.7), turned to -90 degrees
- moved C7 4.41 mm to (116.0, 114.0), turned to -90 degrees
- moved SW2 2.96 mm to (93.8, 103.8)
- moved R8 2.11 mm to (167.7, 92.9), turned to 90 degrees
- moved D3 1.79 mm to (165.8, 84.2), turned to -90 degrees
- moved SW1 1.58 mm to (63.4, 103.8)
- moved R6 1.54 mm to (168.4, 97.4), turned to -90 degrees
- moved R33 1.25 mm to (115.5, 121.6)
- moved R34 1.21 mm to (115.5, 119.2)
- moved SW3 0.64 mm to (76.2, 102.4)
- moved R28 0.37 mm to (115.0, 106.6)
- moved R23 0.31 mm to (116.0, 110.0)
Connections:
- J2 pad 19: /Scv -> (no net)
- J2 pad 20: /Rcv -> (no net)
- J2 pad 21: /EocOut -> (no net)
- J2 pad 22: (no net) -> /Trigger (x2)
- J2 pad 23: /Trigger -> (no net) (x2)
- J2 pad 4: /Acv -> (no net)
- J2 pad 5: /Dcv -> (no net)
- J2 pad 7: (no net) -> Net-(R11-Pad2) (x2)
- J2 pad 4: Net-(R45-Pad2) -> (no net) (x2)
- REF** pad S: (no net) -> GND (x8)
Routing:
- net Net-(R45-Pad2): track 88.0 -> 9.37 mm
- net /Dcv: track 42.0 -> 18.6 mm
- net +12V: track 441.2 -> 418.8 mm
- net Net-(R11-Pad2): track 32.9 -> 54.2 mm
- net /Scv: track 38.5 -> 19.7 mm
- net GND: track 503.3 -> 514.4 mm, vias 1 -> 0
- net Net-(R3-Pad1): track 95.3 -> 85.7 mm
- net Net-(R22-Pad2): track 112.9 -> 105.8 mm
- net Net-(R22-Pad1): track 5.92 -> 10.5 mm
- net Net-(R36-Pad1): track 8.65 -> 5.53 mm
- net /Trigger: track 105.0 -> 102.0 mm
- net /Rcv: track 21.5 -> 18.6 mm
- net /SustainControl: track 39.0 -> 41.9 mm
- net Net-(R24-Pad1): track 48.8 -> 45.8 mm
- net /Vgate: track 93.4 -> 90.5 mm
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Other:
- board size 124.1 x 110.8 mm -> 123.4 x 110.8 mm
